Commit message: Simplified wegde loading uphill/downhill

File: gym_stoch2_sloped_terrain/envs/Wedges/downhill/urdf/wedge_11.urdf (robot description, URDF)
Before this commit: robot Part1, 1 links, 0 joints
Links:
- link ramp_5: geometry collision mesh filename=package://ramp_5/meshes/ramp_5.STL scale=1.5 3.3 1.5; visual mesh filename=package://ramp_5/meshes/ramp_5.STL scale=1.5 3.3 1.5

File: gym_stoch2_sloped_terrain/envs/Wedges/downhill/urdf/wedge_13.urdf (robot description, URDF)
Before this commit: robot Part1, 1 links, 0 joints
Links:
- link ramp_5: geometry collision mesh filename=package://ramp_5/meshes/ramp_5.STL scale=1.5 3.958 1.5; visual mesh filename=package://ramp_5/meshes/ramp_5.STL scale=1.5 3.958 1.5

File: gym_stoch2_sloped_terrain/envs/Wedges/downhill/urdf/wedge_5.urdf (robot description, URDF)
Before this commit: robot Part1, 1 links, 0 joints
Links:
- link ramp_5: geometry collision mesh filename=package://ramp_5/meshes/ramp_5.STL scale=1.5 1.5 1.5; visual mesh filename=package://ramp_5/meshes/ramp_5.STL scale=1.5 1.5 1.5

File: gym_stoch2_sloped_terrain/envs/Wedges/downhill/urdf/wedge_7.urdf (robot description, URDF)
Before this commit: robot Part1, 1 links, 0 joints
Links:
- link ramp_5: geometry collision mesh filename=package://ramp_5/meshes/ramp_5.STL scale=1.5 2.1 1.5; visual mesh filename=package://ramp_5/meshes/ramp_5.STL scale=1.5 2.1 1.5

File: gym_stoch2_sloped_terrain/envs/Wedges/uphill/urdf/wedge_11.urdf (robot description, URDF)
Before this commit: robot Part1, 1 links, 0 joints
Links:
- link ramp_5: geometry collision mesh filename=package://ramp_5/meshes/ramp_5.STL scale=1.5 3.3 1.5; visual mesh filename=package://ramp_5/meshes/ramp_5.STL scale=1.5 3.3 1.5

File: gym_stoch2_sloped_terrain/envs/Wedges/uphill/urdf/wedge_13.urdf (robot description, URDF)
Before this commit: robot Part1, 1 links, 0 joints
Links:
- link ramp_5: geometry collision mesh filename=package://ramp_5/meshes/ramp_5.STL scale=1.5 3.958 1.5; visual mesh filename=package://ramp_5/meshes/ramp_5.STL scale=1.5 3.958 1.5

File: gym_stoch2_sloped_terrain/envs/Wedges/uphill/urdf/wedge_5.urdf (robot description, URDF)
Before this commit: robot Part1, 1 links, 0 joints
Links:
- link ramp_5: geometry collision mesh filename=package://ramp_5/meshes/ramp_5.STL scale=1.5 1.5 1.5; visual mesh filename=package://ramp_5/meshes/ramp_5.STL scale=1.5 1.5 1.5

File: gym_stoch2_sloped_terrain/envs/Wedges/uphill/urdf/wedge_7.urdf (robot description, URDF)
Before this commit: robot Part1, 1 links, 0 joints
Links:
- link ramp_5: geometry collision mesh filename=package://ramp_5/meshes/ramp_5.STL scale=1.5 2.1 1.5; visual mesh filename=package://ramp_5/meshes/ramp_5.STL scale=1.5 2.1 1.5
